File: hardware/8ch/02_controller.kicad_sch (KiCad schematic)
At the start: 0 parts

Commit message: fix bugs
Parts:
- added C49, C50, C51: 100n X7R, Capacitor_SMD:C_0805_2012Metric, symbol Device:C
- added C52: 10n X7R, Capacitor_SMD:C_0805_2012Metric, symbol Device:C
- added J2: LCD_16x2_HEADER, Connector_PinHeader_2.54mm:PinHeader_1x16_P2.54mm_Vertical, symbol Connector_Generic:Conn_01x16
- added J5: AVR_ISP, Connector_PinHeader_2.54mm:PinHeader_2x03_P2.54mm_Vertical, symbol Connector_Generic:Conn_02x03_Odd_Even
- added J6: MCU_EXPANSION, Connector_PinHeader_2.54mm:PinHeader_2x05_P2.54mm_Vertical, symbol Connector_Generic:Conn_02x05_Odd_Even
- added R28: 10k, Resistor_SMD:R_0805_2012Metric, symbol Device:R
- added R29: 220R, Resistor_SMD:R_0805_2012Metric, symbol Device:R
- added RV1: 10k LCD CONTRAST, Potentiometer_THT:Potentiometer_Bourns_3296W_Vertical, symbol Device:R_Potentiometer
- added SW1: NEXT, Button_Switch_THT:SW_PUSH_6mm, symbol Switch:SW_Push
- added SW2: UP, Button_Switch_THT:SW_PUSH_6mm, symbol Switch:SW_Push
- added SW3: DOWN, Button_Switch_THT:SW_PUSH_6mm, symbol Switch:SW_Push
- added SW4: SET, Button_Switch_THT:SW_PUSH_6mm, symbol Switch:SW_Push
- added SW5: ACK, Button_Switch_THT:SW_PUSH_6mm, symbol Switch:SW_Push
- added TP7: RESET_N, TestPoint:TestPoint_THTPad_D2.0mm_Drill1.0mm, symbol Connector_Generic:Conn_01x01
- added U1: ATmega32A-PU, Package_DIP:DIP-40_W15.24mm_Socket, symbol MCU_Microchip_ATmega:ATmega16L-8P
Connections:
- new net +5V_CTRL: C49.1, C49.2, C50.1, C50.2, C51.1, C51.2, C52.1, C52.2, J2.1 (Pin_1), J2.11 (Pin_11), J2.12 (Pin_12), J2.13 (Pin_13), J2.14 (Pin_14), J2.15 (Pin_15), J2.16 (Pin_16), J2.2 (Pin_2), J2.3 (Pin_3), J2.4 (Pin_4), J2.5 (Pin_5), J2.6 (Pin_6), J5.1 (Pin_1), J5.2 (Pin_2), J5.3 (Pin_3), J5.4 (Pin_4), J5.5 (Pin_5), J5.6 (Pin_6), J6.1 (Pin_1), J6.10 (Pin_10), J6.2 (Pin_2), J6.3 (Pin_3), J6.4 (Pin_4), J6.5 (Pin_5), J6.6 (Pin_6), J6.7 (Pin_7), J6.8 (Pin_8), J6.9 (Pin_9), R28.1, R28.2, R29.1, R29.2, RV1.1, RV1.2, RV1.3, SW1.1, SW1.2, SW2.1, SW2.2, SW3.1, SW3.2, SW4.1, SW4.2, SW5.1, SW5.2, TP7.1 (Pin_1), U1.10 (VCC), U1.11 (GND), U1.16 (PD2), U1.17 (PD3), U1.18 (PD4), U1.19 (PD5), U1.20 (PD6), U1.24 (PC2), U1.25 (PC3), U1.26 (PC4), U1.27 (PC5), U1.30 (AVCC), U1.31 (GND), U1.32 (AREF), U1.33 (PA7), U1.34 (PA6), U1.35 (PA5), U1.36 (PA4), U1.37 (PA3), U1.38 (PA2), U1.39 (PA1), U1.40 (PA0), U1.6 (PB5), U1.7 (PB6), U1.8 (PB7), U1.9 (~{RESET})
- new net CS1_CTRL: U1.1 (PB0)
- new net CS2_CTRL: U1.2 (PB1)
- new net CS3_CTRL: U1.3 (PB2)
- new net CS4_CTRL: U1.5 (PB4)
- new net CS5_CTRL: U1.22 (PC0)
- new net CS6_CTRL: U1.23 (PC1)
- new net CS7_CTRL: U1.28 (PC6)
- new net CS8_CTRL: U1.29 (PC7)
- new net RS485_DE: U1.21 (PD7)
- new net RUN_PERMIT: U1.4 (PB3)
- new net UART_RX: U1.14 (PD0)
- new net UART_TX: U1.15 (PD1)
- no-connect marks 0 -> 6
Other:
- removed sheet Channels 1 4
- removed sheet Channels 5 8
- removed sheet Controller
- removed sheet Isolation
- removed sheet Power
- removed sheet Relay
- removed sheet Rs485
- note added: "CONTROLLER"
