File: hardware/8ch/03_channels_1_4.kicad_sch (KiCad schematic)
At the start: 0 parts

Commit message: fix bugs
Parts:
- added C1, C11, C16, C6: 100n C0G 50V, Capacitor_SMD:C_0805_2012Metric, symbol Device:C
- added C10, C14, C15, C19, C20, C4, C5, C9: 100n X7R, Capacitor_SMD:C_0805_2012Metric, symbol Device:C
- added C12, C13, C17, C18, C2, C3, C7, C8: 10n C0G 50V, Capacitor_SMD:C_0805_2012Metric, symbol Device:C
- added JTC1: TC1_K_TYPE, TerminalBlock_Phoenix:TerminalBlock_Phoenix_MKDS-1,5-3_1x03_P5.00mm_Horizontal, symbol Connector_Generic:Conn_01x03
- added JTC2: TC2_K_TYPE, TerminalBlock_Phoenix:TerminalBlock_Phoenix_MKDS-1,5-3_1x03_P5.00mm_Horizontal, symbol Connector_Generic:Conn_01x03
- added JTC3: TC3_K_TYPE, TerminalBlock_Phoenix:TerminalBlock_Phoenix_MKDS-1,5-3_1x03_P5.00mm_Horizontal, symbol Connector_Generic:Conn_01x03
- added JTC4: TC4_K_TYPE, TerminalBlock_Phoenix:TerminalBlock_Phoenix_MKDS-1,5-3_1x03_P5.00mm_Horizontal, symbol Connector_Generic:Conn_01x03
- added R1, R2, R3, R4, R5, R6, R7, R8: 100R 0.1%, Resistor_SMD:R_0805_2012Metric, symbol Device:R
- added R17, R18, R19, R20: 10k, Resistor_SMD:R_0805_2012Metric, symbol Device:R
- added R45, R46, R47, R48: 100R, Resistor_SMD:R_0805_2012Metric, symbol Device:R
- added U2, U3, U4, U5: MAX31856MUD+, Package_SO:TSSOP-14_4.4x5mm_P0.65mm, symbol Sensor_Temperature:MAX31856
Connections:
- new net +3V3_SENS: C10.1, C14.1, C15.1, C19.1, C20.1, C4.1, C5.1, C9.1, R17.1, R18.1, R19.1, R20.1, U2.5 (AVDD), U2.8 (DVDD), U3.5 (AVDD), U3.8 (DVDD), U4.5 (AVDD), U4.8 (DVDD), U5.5 (AVDD), U5.8 (DVDD)
- new net CHASSIS_SHIELD: JTC1.3 (Pin_3), JTC2.3 (Pin_3), JTC3.3 (Pin_3), JTC4.3 (Pin_3)
- new net CS1_SENS: C1.2, C10.2, C11.2, C12.2, C13.1, C13.2, C14.2, C15.2, C16.2, C17.2, C18.1, C18.2, C19.2, C2.2, C20.2, C3.1, C3.2, C4.2, C5.2, C6.2, C7.2, C8.1, C8.2, C9.2, R17.2, R18.2, R19.2, R2.2, R20.2, R4.2, R6.2, R8.2, U2.1 (AGND), U2.12 (SDI), U2.14 (DGND), U2.2 (BIAS), U2.3 (T-), U2.9 (~{CS}), U3.1 (AGND), U3.12 (SDI), U3.14 (DGND), U3.2 (BIAS), U3.3 (T-), U3.9 (~{CS}), U4.1 (AGND), U4.12 (SDI), U4.14 (DGND), U4.2 (BIAS), U4.3 (T-), U4.9 (~{CS}), U5.1 (AGND), U5.12 (SDI), U5.14 (DGND), U5.2 (BIAS), U5.3 (T-), U5.9 (~{CS})
- new net MISO_CH1: R45.1, U2.11 (SDO)
- new net MISO_CH2: R46.1, U3.11 (SDO)
- new net MISO_CH3: R47.1, U4.11 (SDO)
- new net MISO_CH4: R48.1, U5.11 (SDO)
- new net MISO_SENS: R45.2, R46.2, R47.2, R48.2
- new net SCK_SENS: U2.10 (SCK), U3.10 (SCK), U4.10 (SCK), U5.10 (SCK)
- new net TC1_FILT_P: C1.1, C2.1, R1.2, U2.4 (T+)
- new net TC1_RAW_N: JTC1.2 (Pin_2), R2.1
- new net TC1_RAW_P: JTC1.1 (Pin_1), R1.1
- new net TC2_FILT_P: C6.1, C7.1, R3.2, U3.4 (T+)
- new net TC2_RAW_N: JTC2.2 (Pin_2), R4.1
- new net TC2_RAW_P: JTC2.1 (Pin_1), R3.1
- new net TC3_FILT_P: C11.1, C12.1, R5.2, U4.4 (T+)
- new net TC3_RAW_N: JTC3.2 (Pin_2), R6.1
- new net TC3_RAW_P: JTC3.1 (Pin_1), R5.1
- new net TC4_FILT_P: C16.1, C17.1, R7.2, U5.4 (T+)
- new net TC4_RAW_N: JTC4.2 (Pin_2), R8.1
- new net TC4_RAW_P: JTC4.1 (Pin_1), R7.1
- no-connect marks 0 -> 12
Other:
- removed sheet Channels 1 4
- removed sheet Channels 5 8
- removed sheet Controller
- removed sheet Isolation
- removed sheet Power
- removed sheet Relay
- removed sheet Rs485
- note added: "CHANNELS 1 4"
