File: hardware/8ch/05_digital_isolation.kicad_sch (KiCad schematic)
At the start: 0 parts

Commit message: fix bugs
Parts:
- added C41, C42, C43, C44: 100n X7R, Capacitor_SMD:C_0805_2012Metric, symbol Device:C
- added R25, R26, R27: 33R, Resistor_SMD:R_0805_2012Metric, symbol Device:R
- added R36, R37, R38, R39, R40, R41, R42, R43: 22R, Resistor_SMD:R_0805_2012Metric, symbol Device:R
- added TP5: SCK_SENS, TestPoint:TestPoint_THTPad_D2.0mm_Drill1.0mm, symbol Connector_Generic:Conn_01x01
- added TP6: MISO_SENS, TestPoint:TestPoint_THTPad_D2.0mm_Drill1.0mm, symbol Connector_Generic:Conn_01x01
- added U10: ISO7760FDWR, Package_SO:SOIC-16W_7.5x10.3mm_P1.27mm, symbol Isolator:ISO7760DW
- added U11: ISO7761FDWR, Package_SO:SOIC-16W_7.5x10.3mm_P1.27mm, symbol Isolator:ISO7761DW
Connections:
- new net +3V3_SENS: C42.1, C44.1, U10.16 (Vcc2), U11.16 (Vcc2)
- new net +5V_CTRL: C41.1, C43.1, U10.1 (Vcc1), U11.1 (Vcc1)
- new net CS1_CTRL: U10.4 (INC)
- new net CS1_SENS: R36.2
- new net CS1_SENS_RAW: R26.1, R36.1, R37.1, R38.1, R39.1, U10.10 (OUTF), U10.11 (OUTE), U10.12 (OUTD), U10.13 (OUTC), U10.14 (OUTB)
- new net CS2_CTRL: U10.5 (IND)
- new net CS2_SENS: R37.2
- new net CS3_CTRL: U10.6 (INE)
- new net CS3_SENS: R38.2
- new net CS4_CTRL: U10.7 (INF)
- new net CS4_SENS: R39.2
- new net CS5_CTRL: U11.2 (INA)
- new net CS5_SENS: R40.2
- new net CS5_SENS_RAW: R40.1, U11.15 (OUTA)
- new net CS6_CTRL: U11.3 (INB)
- new net CS6_SENS: R41.2
- new net CS6_SENS_RAW: R41.1, U11.14 (OUTB)
- new net CS7_CTRL: U11.4 (INC)
- new net CS7_SENS: R42.2
- new net CS7_SENS_RAW: R42.1, R43.1, U11.12 (OUTD), U11.13 (OUTC)
- new net CS8_CTRL: U11.5 (IND)
- new net CS8_SENS: R43.2
- new net GND_CTRL: C41.2, C42.2, C43.2, C44.2, U10.8 (GND1), U10.9 (GND2), U11.6 (INE), U11.8 (GND1), U11.9 (GND2)
- new net MISO_CTRL: U11.7 (OUTF)
- new net MISO_SENS: R27.1, R27.2, TP6.1 (Pin_1), U11.10 (INF)
- new net MOSI_CTRL: U10.3 (INB)
- new net MOSI_SENS: R26.2
- new net SCK_CTRL: U10.2 (INA)
- new net SCK_SENS: R25.2, TP5.1 (Pin_1)
- new net SCK_SENS_RAW: R25.1, U10.15 (OUTA)
- no-connect marks 0 -> 1
Other:
- removed sheet Channels 1 4
- removed sheet Channels 5 8
- removed sheet Controller
- removed sheet Isolation
- removed sheet Power
- removed sheet Relay
- removed sheet Rs485
- note added: "ISOLATION"
