File: hardware/8ch/06_rs485.kicad_sch (KiCad schematic)
At the start: 0 parts

Commit message: fix bugs
Parts:
- added C56, C58: 100n X7R, Capacitor_SMD:C_0805_2012Metric, symbol Device:C
- added C57, C59: 10u X7R, Capacitor_SMD:C_0805_2012Metric, symbol Device:C
- added D5, D6: SMAJ6.0CA, Diode_SMD:D_SMA, symbol Device:D_TVS
- added J4: RS485_A_B_GND_SHIELD, TerminalBlock_Phoenix:TerminalBlock_Phoenix_MKDS-1,5-4_1x04_P5.00mm_Horizontal, symbol Connector_Generic:Conn_01x04
- added JP1: TERM_ENABLE, Connector_PinHeader_2.54mm:PinHeader_1x02_P2.54mm_Vertical, symbol Connector_Generic:Conn_01x02
- added JP2: BIAS_A_ENABLE, Connector_PinHeader_2.54mm:PinHeader_1x02_P2.54mm_Vertical, symbol Connector_Generic:Conn_01x02
- added JP3: BIAS_B_ENABLE, Connector_PinHeader_2.54mm:PinHeader_1x02_P2.54mm_Vertical, symbol Connector_Generic:Conn_01x02
- added R33: 0R, Resistor_SMD:R_0805_2012Metric, symbol Device:R
- added R34: 120R 1%, Resistor_SMD:R_0805_2012Metric, symbol Device:R
- added R35, R44: 680R 1%, Resistor_SMD:R_0805_2012Metric, symbol Device:R
- added TP8: RS485_A, TestPoint:TestPoint_THTPad_D2.0mm_Drill1.0mm, symbol Connector_Generic:Conn_01x01
- added TP9: RS485_B, TestPoint:TestPoint_THTPad_D2.0mm_Drill1.0mm, symbol Connector_Generic:Conn_01x01
- added U15: ADM2587EBRWZ, Package_SO:SOIC-20W_7.5x12.8mm_P1.27mm, symbol Interface_UART:ADM2587E
Connections:
- new net +5V_CTRL: C56.1, C57.1, U15.2 (VCC), U15.8 (VCC)
- new net +5V_RS485: C58.1, C58.2, C59.1, C59.2, D5.1 (A1), D5.2 (A2), D6.1 (A1), D6.2 (A2), J4.1 (Pin_1), J4.2 (Pin_2), J4.3 (Pin_3), J4.4 (Pin_4), JP1.1 (Pin_1), JP1.2 (Pin_2), JP2.1 (Pin_1), JP2.2 (Pin_2), JP3.1 (Pin_1), JP3.2 (Pin_2), R34.1, R34.2, R35.1, R35.2, R44.1, R44.2, TP8.1 (Pin_1), TP9.1 (Pin_1), U15.11 (GND2), U15.12 (Visoout), U15.13 (Y), U15.14 (GND2), U15.15 (Z), U15.16 (GND2), U15.17 (B), U15.18 (A), U15.19 (Visoin), U15.20 (GND2)
- new net GND_CTRL: C56.2, C57.2, U15.1 (GND1), U15.10 (GND1), U15.3 (GND1), U15.9 (GND1)
- new net RS485_DE: R33.1, R33.2, U15.5 (~{RE}), U15.6 (DE)
- new net UART_RX: U15.4 (RxD)
- new net UART_TX: U15.7 (TxD)
Other:
- removed sheet Channels 1 4
- removed sheet Channels 5 8
- removed sheet Controller
- removed sheet Isolation
- removed sheet Power
- removed sheet Relay
- removed sheet Rs485
- note added: "RS485"
