File: hardware/8ch/thermocouple_8ch.kicad_sch (KiCad schematic)
At the start: 201 parts, among them J1 24V_INPUT, J2 LCD_16x2_HEADER, J3 RELAY_COM_NO_NC, J4 RS485_A_B_GND_SHIELD, J5 AVR_ISP, J6 MCU_EXPANSION, K1 G5LE-1 DC24, Q1 2N7000, SW1 NEXT, SW2 UP, SW3 DOWN, SW4 SET, SW5 ACK, U1 ATmega32A-PU, U10 ISO7760FDWR, U11 ISO7761FDWR, U12 IA0505S, U13 LP2985-3.3, U14 LM5164DDAR, U15 ADM2587EBRWZ, U2 MAX31856MUD+, U3 MAX31856MUD+, U4 MAX31856MUD+, U5 MAX31856MUD+, U6 MAX31856MUD+, U7 MAX31856MUD+, U8 MAX31856MUD+, U9 MAX31856MUD+, Y1 8MHz 20pF

Commit message: Hierarchical schematic; U12 decoupling fixed; two blind gates fixed (I-062, I-045)
Schematic (I-062, decision 0019): an A3 root plus channel.kicad_sch (A4)
used by sheets TC1-TC8, derived by sch_layout/hier.py as the last step of
build.py. Only channel-internal nets were renamed (/TCn_X -> /TCn/X, 40
nets); JTC1-8 value -> K_TYPE (KiCad 10 keeps one value per symbol).
netlist_fingerprint.py --allow-renames proved all 645 pins on the same
nets; the baseline was regenerated from that netlist with the reason in it.
apply_rules.py patterns follow (without them: 499 isolation violations on a
test copy); board nets renamed in place by rename_board_nets.py.

Board (I-045): C45, U12's input cap, sat 55 mm away beside U10; C45/C46 now
sit under U12's pins, 18/10 mm -> 4.2 mm. Re-routed.

Gates that passed on the wrong input: close_gaps.py read a 2026-09-07 DRC
report (now runs its own with --refill-zones); check_mpn_consistency.py read
only the root after the split, 56 of 128 symbols (now follows every sheet
and runs inside validate.ps1, I-054 downgraded). populate_schematic.py
refuses the hierarchical root.

validate.ps1, KiCad 10.0.6: ERC 0/0, netlist IDENTICAL 201/162/645, MPN
128/128, DRC 0 errors / 0 warnings / 0 unconnected / 0 parity.
check_board.py all 6 ok. firmware/build.ps1: 3 suites pass.

Co-Authored-By: Claude Opus 5.5 <noreply@anthropic.com>
Parts:
- removed C1, C11, C16, C21, C26, C31, C36, C6: 100n X7R 50V, Capacitor_SMD:C_0805_2012Metric, symbol Device:C
- removed C10, C14, C15, C19, C20, C24, C25, C29, C30, C34, C35, C39, C4, C40, C5, C9: 100n X7R, Capacitor_SMD:C_0805_2012Metric, symbol Device:C
- removed C12, C13, C17, C18, C2, C22, C23, C27, C28, C3, C32, C33, C37, C38, C7, C8: 10n C0G 50V, Capacitor_SMD:C_0805_2012Metric, symbol Device:C
- removed D10, D11, D12, D13, D14, D15, D16, D17, D18, D19, D20, D21, D22, D7, D8, D9: BAV199, Package_TO_SOT_SMD:SOT-23, symbol Device:D_Dual_Series_AKC
- removed JTC1: TC1_K_TYPE, TerminalBlock_Phoenix:TerminalBlock_Phoenix_MKDS-1,5-3_1x03_P5.00mm_Horizontal, symbol Connector_Generic:Conn_01x03
- removed JTC2: TC2_K_TYPE, TerminalBlock_Phoenix:TerminalBlock_Phoenix_MKDS-1,5-3_1x03_P5.00mm_Horizontal, symbol Connector_Generic:Conn_01x03
- removed JTC3: TC3_K_TYPE, TerminalBlock_Phoenix:TerminalBlock_Phoenix_MKDS-1,5-3_1x03_P5.00mm_Horizontal, symbol Connector_Generic:Conn_01x03
- removed JTC4: TC4_K_TYPE, TerminalBlock_Phoenix:TerminalBlock_Phoenix_MKDS-1,5-3_1x03_P5.00mm_Horizontal, symbol Connector_Generic:Conn_01x03
- removed JTC5: TC5_K_TYPE, TerminalBlock_Phoenix:TerminalBlock_Phoenix_MKDS-1,5-3_1x03_P5.00mm_Horizontal, symbol Connector_Generic:Conn_01x03
- removed JTC6: TC6_K_TYPE, TerminalBlock_Phoenix:TerminalBlock_Phoenix_MKDS-1,5-3_1x03_P5.00mm_Horizontal, symbol Connector_Generic:Conn_01x03
- removed JTC7: TC7_K_TYPE, TerminalBlock_Phoenix:TerminalBlock_Phoenix_MKDS-1,5-3_1x03_P5.00mm_Horizontal, symbol Connector_Generic:Conn_01x03
- removed JTC8: TC8_K_TYPE, TerminalBlock_Phoenix:TerminalBlock_Phoenix_MKDS-1,5-3_1x03_P5.00mm_Horizontal, symbol Connector_Generic:Conn_01x03
- removed R1, R10, R11, R12, R13, R14, R15, R16, R2, R3, R4, R5, R6, R7, R8, R9: 100R 0.1%, Resistor_SMD:R_0805_2012Metric, symbol Device:R
- removed R17, R18, R19, R20, R21, R22, R23, R24: 10k, Resistor_SMD:R_0805_2012Metric, symbol Device:R
- removed R45, R46, R47, R48, R49, R50, R51, R52: 100R, Resistor_SMD:R_0805_2012Metric, symbol Device:R
- removed U2, U3, U4, U5, U6, U7, U8, U9: MAX31856MUD+, Package_SO:TSSOP-14_4.4x5mm_P0.65mm, symbol Sensor_Temperature:MAX31856
Connections:
- no-connect marks 33 -> 9
Other:
- added sheet TC1 (channel.kicad_sch)
- added sheet TC2 (channel.kicad_sch)
- added sheet TC3 (channel.kicad_sch)
- added sheet TC4 (channel.kicad_sch)
- added sheet TC5 (channel.kicad_sch)
- added sheet TC6 (channel.kicad_sch)
- added sheet TC7 (channel.kicad_sch)
- added sheet TC8 (channel.kicad_sch)
- moved on the sheet: C41, C42, C43, C44, C45, C46, C47, C48, C49, C50, C51, C52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

Commit message: Schematic on six A4 sheets by function (0021); external panel fuse specified (0020)
The root's remaining blocks move to power, mcu, isolation and relay_rs485
sheets; the root becomes an A4 index beside the reused channel sheet.
56 sheet-internal nets gain the sheet path. apply_rules.py patterns and
board/units.bare() follow, and all 162 board nets keep their netclass.
Board nets renamed in place, copper unchanged. validate.ps1: ERC 0/0,
netlist IDENTICAL, MPN 128/128, DRC 0/0/0/0; check_board all ok; build.py
reproduces the six sheets.

I-028 (a): external 1 A time-delay DC fuse, >= 80 V DC, >= 10 kA, at the
battery end; inrush in CALCULATIONS.md 1.9. New low I-064 (board overlaps
its PCB-editor page frame, cosmetic).

Co-Authored-By: Claude Opus 5.5 <noreply@anthropic.com>
Parts:
- removed C41, C42, C43, C44, C49, C50, C51, C56, C58: 100n X7R, Capacitor_SMD:C_0805_2012Metric, symbol Device:C
- removed C45, C46: 10u 10V, Capacitor_SMD:C_0805_2012Metric, symbol Device:C
- removed C47: 1u X7R, Capacitor_SMD:C_0805_2012Metric, symbol Device:C
- removed C48: 4.7u X7R 16V, Capacitor_SMD:C_0805_2012Metric, symbol Device:C
- removed C52: 10n X7R, Capacitor_SMD:C_0805_2012Metric, symbol Device:C
- removed C53: 22u 100V, Capacitor_THT:CP_Radial_D8.0mm_P3.50mm, symbol Device:C
- removed C54, C63: 4.7u 100V X7R, Capacitor_SMD:C_1210_3225Metric, symbol Device:C
- removed C55: 10u 10V X7R, Capacitor_SMD:C_0805_2012Metric, symbol Device:C
- removed C57, C59: 10u X7R, Capacitor_SMD:C_0805_2012Metric, symbol Device:C
- removed C60, C61: 22p C0G 50V, Capacitor_SMD:C_0805_2012Metric, symbol Device:C
- removed C62: 2.2n 50V X7R, Capacitor_SMD:C_0805_2012Metric, symbol Device:C
- removed C64, C65: 22u 25V X7R, Capacitor_SMD:C_1210_3225Metric, symbol Device:C
- removed C67: 3.3n 50V X7R, Capacitor_SMD:C_0805_2012Metric, symbol Device:C
- removed C68: 220p C0G 50V, Capacitor_SMD:C_0805_2012Metric, symbol Device:C
- removed D1: SS310, Diode_SMD:D_SMA, symbol Device:D_Schottky
- removed D2: SMBJ60A, Diode_SMD:D_SMB, symbol Device:D_TVS
- removed D3: 1N4007, Diode_SMD:D_SMA, symbol Device:D
- removed D4: RUN PERMIT, LED_THT:LED_D3.0mm, symbol Device:LED
- removed D5, D6: SMAJ6.0CA, Diode_SMD:D_SMA, symbol Device:D_TVS
- removed F1: PTC 0.5A, Fuse:Fuse_1206_3216Metric, symbol Device:Polyfuse
- removed J1: 24V_INPUT, TerminalBlock_Phoenix:TerminalBlock_Phoenix_MKDS-1,5-3_1x03_P5.00mm_Horizontal, symbol Connector_Generic:Conn_01x03
- removed J2: LCD_16x2_HEADER, Connector_PinHeader_2.54mm:PinHeader_1x16_P2.54mm_Vertical, symbol Connector_Generic:Conn_01x16
- removed J3: RELAY_COM_NO_NC, TerminalBlock_Phoenix:TerminalBlock_Phoenix_MKDS-1,5-3_1x03_P5.00mm_Horizontal, symbol Connector_Generic:Conn_01x03
- removed J4: RS485_A_B_GND_SHIELD, TerminalBlock_Phoenix:TerminalBlock_Phoenix_MKDS-1,5-4_1x04_P5.00mm_Horizontal, symbol Connector_Generic:Conn_01x04
- removed J5: AVR_ISP, Connector_PinHeader_2.54mm:PinHeader_2x03_P2.54mm_Vertical, symbol Connector_Generic:Conn_02x03_Odd_Even
- removed J6: MCU_EXPANSION, Connector_PinHeader_2.54mm:PinHeader_2x05_P2.54mm_Vertical, symbol Connector_Generic:Conn_02x05_Odd_Even
- removed JP1: TERM_ENABLE, Connector_PinHeader_2.54mm:PinHeader_1x02_P2.54mm_Vertical, symbol Connector_Generic:Conn_01x02
- removed JP2: BIAS_A_ENABLE, Connector_PinHeader_2.54mm:PinHeader_1x02_P2.54mm_Vertical, symbol Connector_Generic:Conn_01x02
- removed JP3: BIAS_B_ENABLE, Connector_PinHeader_2.54mm:PinHeader_1x02_P2.54mm_Vertical, symbol Connector_Generic:Conn_01x02
- removed K1: G5LE-1 DC24, Relay_THT:Relay_SPDT_Omron-G5LE-1, symbol Relay:G5LE-1
- removed L1: 33u 2.2A, Inductor_SMD:L_10.4x10.4_H4.8, symbol Device:L
- removed Q1: 2N7000, Package_TO_SOT_THT:TO-92_Inline_Wide, symbol Transistor_FET:2N7000
- removed R25, R26, R27: 33R, Resistor_SMD:R_0805_2012Metric, symbol Device:R
- removed R28: 10k, Resistor_SMD:R_0805_2012Metric, symbol Device:R
- removed R29: 220R, Resistor_SMD:R_0805_2012Metric, symbol Device:R
- removed R30: 100R, Resistor_SMD:R_0805_2012Metric, symbol Device:R
- removed R31: 100k, Resistor_SMD:R_0805_2012Metric, symbol Device:R
- removed R32: 4.7k 0.25W, Resistor_SMD:R_0805_2012Metric, symbol Device:R
- removed R33: 0R, Resistor_SMD:R_0805_2012Metric, symbol Device:R
- removed R34: 120R 1%, Resistor_SMD:R_0805_2012Metric, symbol Device:R
- removed R35, R44: 680R 1%, Resistor_SMD:R_0805_2012Metric, symbol Device:R
- removed R36, R37, R38, R39, R40, R41, R42, R43: 22R, Resistor_SMD:R_0805_2012Metric, symbol Device:R
- removed R53: 22k, Resistor_SMD:R_0805_2012Metric, symbol Device:R
- removed R54: 4k7, Resistor_SMD:R_0805_2012Metric, symbol Device:R
- removed R55: 41.2k 1%, Resistor_SMD:R_0805_2012Metric, symbol Device:R
- removed R56: 158k 1%, Resistor_SMD:R_0805_2012Metric, symbol Device:R
- removed R57: 49.9k 1%, Resistor_SMD:R_0805_2012Metric, symbol Device:R
- removed R58: 150k 1%, Resistor_SMD:R_0805_2012Metric, symbol Device:R
- removed R59: 33.2k 1%, Resistor_SMD:R_0805_2012Metric, symbol Device:R
- removed R60: 10k 1%, Resistor_SMD:R_0805_2012Metric, symbol Device:R
- removed RV1: 10k LCD CONTRAST, Potentiometer_THT:Potentiometer_Bourns_3296W_Vertical, symbol Device:R_Potentiometer
- removed SW1: NEXT, Button_Switch_THT:SW_PUSH_6mm, symbol Switch:SW_Push
- removed SW2: UP, Button_Switch_THT:SW_PUSH_6mm, symbol Switch:SW_Push
- removed SW3: DOWN, Button_Switch_THT:SW_PUSH_6mm, symbol Switch:SW_Push
- removed SW4: SET, Button_Switch_THT:SW_PUSH_6mm, symbol Switch:SW_Push
- removed SW5: ACK, Button_Switch_THT:SW_PUSH_6mm, symbol Switch:SW_Push
- removed TP1: GND_CTRL, TestPoint:TestPoint_THTPad_D2.0mm_Drill1.0mm, symbol Connector_Generic:Conn_01x01
- removed TP2: +5V_CTRL, TestPoint:TestPoint_THTPad_D2.0mm_Drill1.0mm, symbol Connector_Generic:Conn_01x01
- removed TP3: GND_SENS, TestPoint:TestPoint_THTPad_D2.0mm_Drill1.0mm, symbol Connector_Generic:Conn_01x01
- removed TP4: +3V3_SENS, TestPoint:TestPoint_THTPad_D2.0mm_Drill1.0mm, symbol Connector_Generic:Conn_01x01
- removed TP5: SCK_SENS, TestPoint:TestPoint_THTPad_D2.0mm_Drill1.0mm, symbol Connector_Generic:Conn_01x01
- removed TP6: MISO_SENS, TestPoint:TestPoint_THTPad_D2.0mm_Drill1.0mm, symbol Connector_Generic:Conn_01x01
- removed TP7: RESET_N, TestPoint:TestPoint_THTPad_D2.0mm_Drill1.0mm, symbol Connector_Generic:Conn_01x01
- removed TP8: RS485_A, TestPoint:TestPoint_THTPad_D2.0mm_Drill1.0mm, symbol Connector_Generic:Conn_01x01
- removed TP9: RS485_B, TestPoint:TestPoint_THTPad_D2.0mm_Drill1.0mm, symbol Connector_Generic:Conn_01x01
- removed U1: ATmega32A-PU, Package_DIP:DIP-40_W15.24mm_Socket, symbol MCU_Microchip_ATmega:ATmega16L-8P
- removed U10: ISO7760FDWR, Package_SO:SOIC-16W_7.5x10.3mm_P1.27mm, symbol Isolator:ISO7760DW
- removed U11: ISO7761FDWR, Package_SO:SOIC-16W_7.5x10.3mm_P1.27mm, symbol Isolator:ISO7761DW
- removed U12: IA0505S, Converter_DCDC:Converter_DCDC_XP_POWER-IAxxxxS_THT, symbol Converter_DCDC_Isolated:IA0505S
- removed U13: LP2985-3.3, Package_TO_SOT_SMD:SOT-23-5, symbol Regulator_Linear:LP2985-1.8
- removed U14: LM5164DDAR, Package_SO:SOIC-8-1EP_3.9x4.9mm_P1.27mm_EP2.41x3.3mm_ThermalVias, symbol Regulator_Switching:LM5164DDA
- removed U15: ADM2587EBRWZ, Package_SO:SOIC-20W_7.5x12.8mm_P1.27mm, symbol Interface_UART:ADM2587E
- removed Y1: 8MHz 20pF, Crystal:Crystal_SMD_HC49-SD, symbol Device:Crystal
Connections:
- no-connect marks 9 -> 0
Other:
- added sheet ISOLATION (isolation.kicad_sch)
- added sheet MCU (mcu.kicad_sch)
- added sheet POWER (power.kicad_sch)
- added sheet RELAY_RS485 (relay_rs485.kicad_sch)
