File: hardware/8ch/thermocouple_8ch.kicad_pcb (KiCad board)
At the start: 4 copper layers, 250 x 140 mm, 174 parts, among them J1 24V_INPUT, J2 LCD_16x2_HEADER, J3 RELAY_COM_NO_NC, J4 RS485_A_B_GND_SHIELD, J5 AVR_ISP, J6 MCU_EXPANSION, K1 G5LE-1 DC24, Q1 2N7000, SW1 NEXT, SW2 UP, SW3 DOWN, SW4 SET, SW5 ACK, U1 ATmega32A-PU, U10 ISO7760FDWR, U11 ISO7761FDWR, U12 IA0505S, U13 LP2985-3.3, U14 TSR 1-2450, U15 ADM2587EBRWZ, U2 MAX31856MUD+, U3 MAX31856MUD+, U4 MAX31856MUD+, U5 MAX31856MUD+, U6 MAX31856MUD+, U7 MAX31856MUD+, U8 MAX31856MUD+, U9 MAX31856MUD+

Commit message: REV A1 board regenerated and routed (I-061, I-060)
Owner decisions: keep U14's 0.2 mm thermal vias and lower the board hole
minimum (0017); J3 keeps COM/NO/NC and moves to line up with K1 (0018).

Fixed on the way:
- R59/R60 turned to 270 so R60's GND pad is not walled in by routing.
- MAX31856 GND pins get fixed vias like the supply pins; left to the pour,
  one floated per run (U3.14, then U5.14).
- route.py re-stitches pour pieces after closing gaps.

Measured with KiCad 10.0.3: check_board.py all 6 ok; DRC with zone refill
and schematic parity: 0 errors, 0 unconnected, 0 parity, 14 silkscreen
warnings. validate.ps1 stops at ERC on I-063 (KiCad version), not the board.

Co-Authored-By: Claude Opus 5.5 <noreply@anthropic.com>
Parts:
- added C60: 22p C0G 50V, Capacitor_SMD:C_0805_2012Metric, F.Cu at (203.7, 71.5)
- added C61: 22p C0G 50V, Capacitor_SMD:C_0805_2012Metric, F.Cu at (195.3, 71.5)
- added C62: 2.2n 50V X7R, Capacitor_SMD:C_0805_2012Metric, F.Cu at (176.5, 105.5)
- added C63: 4.7u 100V X7R, Capacitor_SMD:C_1210_3225Metric, F.Cu at (170.8, 104.5)
- added C64: 22u 25V X7R, Capacitor_SMD:C_1210_3225Metric, F.Cu at (193.5, 108.0)
- added C65: 22u 25V X7R, Capacitor_SMD:C_1210_3225Metric, F.Cu at (197.5, 108.0)
- added C67: 3.3n 50V X7R, Capacitor_SMD:C_0805_2012Metric, F.Cu at (184.5, 102.5)
- added C68: 220p C0G 50V, Capacitor_SMD:C_0805_2012Metric, F.Cu at (172.5, 115.0)
- added D10: BAV199, Package_TO_SOT_SMD:SOT-23, F.Cu at (52.5, 14.2)
- added D11: BAV199, Package_TO_SOT_SMD:SOT-23, F.Cu at (68.5, 14.2)
- added D12: BAV199, Package_TO_SOT_SMD:SOT-23, F.Cu at (82.5, 14.2)
- added D13: BAV199, Package_TO_SOT_SMD:SOT-23, F.Cu at (98.5, 14.2)
- added D14: BAV199, Package_TO_SOT_SMD:SOT-23, F.Cu at (112.5, 14.2)
- added D15: BAV199, Package_TO_SOT_SMD:SOT-23, F.Cu at (29.5, 125.8)
- added D16: BAV199, Package_TO_SOT_SMD:SOT-23, F.Cu at (15.5, 125.8)
- added D17: BAV199, Package_TO_SOT_SMD:SOT-23, F.Cu at (59.5, 125.8)
- added D18: BAV199, Package_TO_SOT_SMD:SOT-23, F.Cu at (45.5, 125.8)
- added D19: BAV199, Package_TO_SOT_SMD:SOT-23, F.Cu at (89.5, 125.8)
- added D20: BAV199, Package_TO_SOT_SMD:SOT-23, F.Cu at (75.5, 125.8)
- added D21: BAV199, Package_TO_SOT_SMD:SOT-23, F.Cu at (119.5, 125.8)
- added D22: BAV199, Package_TO_SOT_SMD:SOT-23, F.Cu at (105.5, 125.8)
- added D7: BAV199, Package_TO_SOT_SMD:SOT-23, F.Cu at (8.50, 14.2)
- added D8: BAV199, Package_TO_SOT_SMD:SOT-23, F.Cu at (22.5, 14.2)
- added D9: BAV199, Package_TO_SOT_SMD:SOT-23, F.Cu at (38.5, 14.2)
- added L1: 33u 2.2A, Inductor_SMD:L_10.4x10.4_H4.8, F.Cu at (185.0, 110.0)
- added R53: 22k, Resistor_SMD:R_0805_2012Metric, F.Cu at (205.5, 103.0)
- added R54: 4k7, Resistor_SMD:R_0805_2012Metric, F.Cu at (205.5, 107.0)
- added R55: 41.2k 1%, Resistor_SMD:R_0805_2012Metric, F.Cu at (167.5, 114.5)
- added R56: 158k 1%, Resistor_SMD:R_0805_2012Metric, F.Cu at (171.5, 117.6)
- added R57: 49.9k 1%, Resistor_SMD:R_0805_2012Metric, F.Cu at (176.3, 115.0)
- added R58: 150k 1%, Resistor_SMD:R_0805_2012Metric, F.Cu at (180.5, 102.5)
- added R59: 33.2k 1%, Resistor_SMD:R_0805_2012Metric, F.Cu at (163.5, 111.0)
- added R60: 10k 1%, Resistor_SMD:R_0805_2012Metric, F.Cu at (163.5, 115.0)
- added Y1: 8MHz 20pF, Crystal:Crystal_SMD_HC49-SD, F.Cu at (199.5, 67.0)
- C1, C11, C16, C21, C26, C31, C36, C6: value 100n C0G 50V -> 100n X7R 50V
- C48: value 1u X7R -> 4.7u X7R 16V
- C53: value 47u 50V -> 22u 100V; footprint Capacitor_THT:CP_Radial_D6.3mm_P2.50mm -> Capacitor_THT:CP_Radial_D8.0mm_P3.50mm
- C54: value 2.2u 50V X7R -> 4.7u 100V X7R; footprint Capacitor_SMD:C_0805_2012Metric -> Capacitor_SMD:C_1210_3225Metric
- D1: value SS34 -> SS310
- D2: value SMBJ33A -> SMBJ60A
- D3: footprint Diode_THT:D_DO-41_SOD81_P10.16mm_Horizontal -> Diode_SMD:D_SMA
- U14: value TSR 1-2450 -> LM5164DDAR; footprint Converter_DCDC:Converter_DCDC_TRACO_TSR-1_THT -> Package_SO:SOIC-8-1EP_3.9x4.9mm_P1.27mm_EP2.41x3.3mm_ThermalVias
- moved U14 27.7 mm to (172.0, 110.0)
- moved C54 27.0 mm to (165.5, 104.5)
- moved C55 17.5 mm to (201.5, 108.0), turned to 90 degrees
- moved R33 8.60 mm to (233.4, 87.0)
- moved J3 7.00 mm to (241.0, 86.0)
- moved C57 6.40 mm to (242.0, 91.0)
- moved C56 2.20 mm to (229.8, 87.0)
Connections:
- J6 pad 3: /SPARE_PC2 -> unconnected-(J6-Pin_3-Pad3)
- K1 pad 1: /RELAY_LOW -> /RELAY_COM
- K1 pad 4: /RELAY_COM -> /RELAY_NC
- K1 pad 5: /RELAY_NC -> /RELAY_LOW
- U1 pad 12: unconnected-(U1-XTAL2-Pad12) -> /XTAL2
- U1 pad 13: unconnected-(U1-XTAL1-Pad13) -> /XTAL1
- U1 pad 24: /SPARE_PC2 -> /RUN_PERMIT_SENSE
- U14 pad 1: /+24V_PROT -> /GND_CTRL
- U14 pad 2: /GND_CTRL -> /+24V_PROT
- U14 pad 3: /+5V_CTRL -> /VIN_UVLO
Routing:
- net /CHASSIS_SHIELD: track 1632.0 -> 816.0 mm
- net /GND_SENS: track 38.0 -> 210.4 mm, vias 7 -> 18
- net /RUN_PERMIT_SENSE: track 0.00 -> 71.8 mm, vias 0 -> 1
- net /SPARE_PC2: track 56.4 -> 0.00 mm, vias 1 -> 0
- net /+3V3_SENS: track 87.0 -> 138.2 mm, vias 38 -> 51
- net /RELAY_COM: track 10.1 -> 39.8 mm
- net /RIPPLE_INJ: track 0.00 -> 29.4 mm
- net /MOSI_SENS: track 348.0 -> 322.8 mm, vias 6 -> 4
- net /MISO_SENS: track 336.4 -> 313.6 mm, vias 7 -> 9
- net /SCK_SENS: track 320.0 -> 342.6 mm, vias 6 -> 11
- net /CS7_SENS: track 99.3 -> 77.8 mm
- net /+5V_CTRL: track 72.7 -> 93.6 mm, vias 5 -> 7
- net /UART_TX: track 44.0 -> 60.1 mm, vias 1 -> 2
- net /SW_5V: track 0.00 -> 14.4 mm
- net /XTAL1: track 0.00 -> 14.1 mm
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