File: hardware/8ch/channel.kicad_sch (KiCad schematic)
At the start: 13 parts, among them U2 MAX31856MUD+

Commit message: Image guard refuses unapproved images (I-082); refused-ACK reason on LCD (I-088); every BOM line sourced (0027)
- program.ps1 exits 2 on any image but thermo_8ch_max31856.hex (run: legacy image -> exit 2, no avrdude)
- NO ACK CHn HOT/FAULT status after a refused ACK; permit logic unchanged
- LCSC codes: MAX31856MUD+T, LP2985, ADM2587E, ATmega32A-PU, 3296W
- substitutes: K1 G5LE-14 DC24, C53 Rubycon 100YXF22; U12 XP IA0505S from DigiKey
- technician fits THT; 3 boards
build.ps1 exit 0, 3 suites PASS; validate.ps1 01:25 ERC 0/0, IDENTICAL, DRC 0/0/0/0.

Co-Authored-By: Claude Opus 5.5 <noreply@anthropic.com>
Parts:
- U2: LCSC (none) -> C2653162; MPN MAX31856MUD+ -> MAX31856MUD+T
Changed lines of the file:
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@@
 			)
 		)
-		(property "MPN" "MAX31856MUD+"
+		(property "MPN" "MAX31856MUD+T"
 			(at 170.18 113.03 0)
 			(hide yes)
@@
 			(effects
 				(font
+					(size 1.27 1.27)
+				)
+			)
+		)
+		(property "LCSC" "C2653162"
+			(at 171.45 107.95 0)
+			(hide yes)
+			(effects
+				(font
