File: hardware/8ch/isolation.kicad_sch (KiCad schematic)
At the start: 27 parts, among them U10 ISO7760FDWR, U11 ISO7761FDWR, U12 IA0505S, U13 LP2985-3.3

Commit message: REV A2: pre-fabrication fixes I-065..I-069 (decision 0022)
- U10/U11 ISO7760DWR/ISO7761DWR (no F: open input -> HIGH) + R61 2k2 on
  U11 OUTF -> MISO_CTRL so in-circuit ISP works (I-065)
- Q1 BSS131 240 V SOT-23 replaces the 60 V 2N7000 (I-066)
- R53/R54 100k/22k: 0.28 mA into PC2's clamp at 58 V (I-067)
- F1 1812L075/60GR, 60 V 0.75 A 1812 (I-068)
- D2 drawn unidirectional, D3 = M7 SMA, U12 sourcing warning (I-069)
- netlist-baseline-reva2.json (202/163/647), BOARD_REV A2
- board regenerated and re-routed; one hand via for C41.1 (+5V_CTRL)
- run_all.ps1 no longer calls populate_schematic.py (hierarchical sheet)

validate.ps1 2026-09-28 01:07: ERC 0/0, netlist IDENTICAL, DRC 0/0/0/0;
check_board.py all 6 ok; firmware build + 3 suites pass.

Co-Authored-By: Claude Opus 5.5 <noreply@anthropic.com>
Parts:
- added R61: 2k2, Resistor_SMD:R_0805_2012Metric, symbol Device:R
- U10: value ISO7760FDWR -> ISO7760DWR; LCSC (none) -> C882724; MPN ISO7760FDWR -> ISO7760DWR
- U11: value ISO7761FDWR -> ISO7761DWR; LCSC (none) -> C2871529; MPN ISO7761FDWR -> ISO7761DWR
Connections:
- net MISO_CTRL: now also R61.1; no longer U11.7 (OUTF)
- new net MISO_ISO: R61.2, U11.7 (OUTF)
Other:
- moved on the sheet: C41, C42, C43, C44, R25, R26, R27, R36, R37, R38, R39, R40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

Commit message: Image guard refuses unapproved images (I-082); refused-ACK reason on LCD (I-088); every BOM line sourced (0027)
- program.ps1 exits 2 on any image but thermo_8ch_max31856.hex (run: legacy image -> exit 2, no avrdude)
- NO ACK CHn HOT/FAULT status after a refused ACK; permit logic unchanged
- LCSC codes: MAX31856MUD+T, LP2985, ADM2587E, ATmega32A-PU, 3296W
- substitutes: K1 G5LE-14 DC24, C53 Rubycon 100YXF22; U12 XP IA0505S from DigiKey
- technician fits THT; 3 boards
build.ps1 exit 0, 3 suites PASS; validate.ps1 01:25 ERC 0/0, IDENTICAL, DRC 0/0/0/0.

Co-Authored-By: Claude Opus 5.5 <noreply@anthropic.com>
Parts:
- U13: LCSC (none) -> C129375
Changed lines of the file:
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@@
+			)
+		)
+		(property "LCSC" "C129375"
+			(at 166.37 146.05 0)
+			(hide yes)
+			(effects
+				(font
+					(size 1.27 1.27)
+				)
 			)
 		)
@@
 			)
 		)
-		(property "Description" "Shared 1 kV functional-isolation supply for the measurement island | Manufacturer: XP Power | MPN: IA0505S - not the regulated 'IA0505S-1WR3' of another maker (I-069)"
+		(property "Description" "Shared 1 kV functional-isolation supply for the measurement island | Manufacturer: XP Power | MPN: IA0505S - not the regulated 'IA0505S-1WR3' of another maker (I-069). Not at LCSC: buy at DigiKey 1470-1345-5-ND, hand-fit (0027)"
 			(at 123.19 146.05 0)
 			(hide yes)
