File: hardware/8ch/mcu.kicad_sch (KiCad schematic)
At the start: 20 parts, among them J2 LCD_16x2_HEADER, J5 AVR_ISP, J6 MCU_EXPANSION, SW1 NEXT, SW2 UP, SW3 DOWN, SW4 SET, SW5 ACK, U1 ATmega32A-PU, Y1 8MHz 20pF

Commit message: Image guard refuses unapproved images (I-082); refused-ACK reason on LCD (I-088); every BOM line sourced (0027)
- program.ps1 exits 2 on any image but thermo_8ch_max31856.hex (run: legacy image -> exit 2, no avrdude)
- NO ACK CHn HOT/FAULT status after a refused ACK; permit logic unchanged
- LCSC codes: MAX31856MUD+T, LP2985, ADM2587E, ATmega32A-PU, 3296W
- substitutes: K1 G5LE-14 DC24, C53 Rubycon 100YXF22; U12 XP IA0505S from DigiKey
- technician fits THT; 3 boards
build.ps1 exit 0, 3 suites PASS; validate.ps1 01:25 ERC 0/0, IDENTICAL, DRC 0/0/0/0.

Co-Authored-By: Claude Opus 5.5 <noreply@anthropic.com>
Parts:
- RV1: LCSC (none) -> C34846
- U1: LCSC (none) -> C12703
Changed lines of the file:
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@@
+			)
+		)
+		(property "LCSC" "C12703"
+			(at 130.81 99.06 0)
+			(hide yes)
+			(effects
+				(font
+					(size 1.27 1.27)
+				)
 			)
 		)
@@
 			(effects
 				(font
+					(size 1.27 1.27)
+				)
+			)
+		)
+		(property "LCSC" "C34846"
+			(at 166.37 35.56 0)
+			(hide yes)
+			(effects
+				(font
