File: hardware/24ch/power.kicad_sch (KiCad schematic)
At the start: 27 parts, among them J601 24V IN, U601 LM5164DDAR

Commit message: 24ch cheaper-parts variant (0036): TMP126, CA-IS3761HW, RS-485 DNP, drop-in swaps
- CJ sensors ADT7310 x6 -> TMP126DCKR (C5219998); R443 22k DIN_ISO-DOUT_ISO for the
  3-wire SIO, R415 removed, ALERT grounded. Sensors moved <= 8 mm to clear spots beside
  their 100 nF (no closer spot to the terminals without touching TC traces, 0035 D2).
- ISO7761 -> CA-IS3761HW (same pinout, 5F/1R, default high); BOCHEN 3296W trimmer;
  SAMWHA 22u 1210.
- RS-485 block DNP: footprints kept; fab.py drops DNP parts from BOM/CPL and writes
  DNP.txt; cost.py skips them. External window watchdog tried and removed (owner).
- gen/delta.py: carry a schematic change onto the routed board (replace/add/remove,
  re-net, DNP, OLD>NEW@DEG reuse); it never deletes another net's track under a pad.
- Board: incremental edits only; analog nets (TC*, V_BIAS, VREF, REF*) identical to
  the pre-0036 board. Gates: ERC 0/0 (471 symbols); fab.py DRC/unconnected/parity
  0/0/0; pincaps 0 over. Parts ~$105 -> ~$72/board (CALCULATIONS 8.1, by hand).
- Docs: decision 0036, CALCULATIONS 8, ISSUES (I-109, I-114, I-119, I-104, I-094,
  new I-123 stock), STATE, 24ch README, superseded.txt.

Co-Authored-By: Claude Opus 5.5 <noreply@anthropic.com>
Parts:
- C605, C606: LCSC C309062 -> C2918511; MPN CL32B226KAJNNNE -> CS3225X7R226K250NRL; Manufacturer (none) -> SAMWHA
Changed lines of the file:
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@@
 			)
 		)
-		(property "MPN" "CL32B226KAJNNNE"
+		(property "MPN" "CS3225X7R226K250NRL"
 			(at 96.52 83.82 0)
 			(effects
@@
 			)
 		)
-		(property "LCSC" "C309062"
+		(property "Manufacturer" "SAMWHA"
+			(at 96.52 83.82 0)
+			(effects
+				(font
+					(size 1.27 1.27)
+				)
+				(hide yes)
+			)
+		)
+		(property "LCSC" "C2918511"
 			(at 96.52 83.82 0)
 			(effects
@@
 			)
 		)
-		(property "MPN" "CL32B226KAJNNNE"
+		(property "MPN" "CS3225X7R226K250NRL"
 			(at 114.3 83.82 0)
 			(effects
@@
 			)
 		)
-		(property "LCSC" "C309062"
+		(property "Manufacturer" "SAMWHA"
 			(at 114.3 83.82 0)
 			(effects
+				(font
+					(size 1.27 1.27)
+				)
+				(hide yes)
+			)
+		)
+		(property "LCSC" "C2918511"
+			(at 114.3 83.82 0)
+			(effects

Commit message: 24ch 0036 D7/D8: screw terminals face the board edge; supplier files as an RFQ
- J601/J701/J702/J703 turned 180 deg about the middle pin (wire entry was blocked by the
  relays ~2 mm in front); pin numbers 1<->3 swapped in the generator so every position keeps
  its net, label and copper. RS-485 row (DNP) moved 0.5 mm with its track ends, BIAS_B routed
  around J703 pin 1, TRIP_COM stub extended to the round pad.
- delta.py: MPN/LCSC/Manufacturer fields go to F.Fab hidden (were printed on the silkscreen of
  the six TMP126), new footprints hide reference/value like the rest of the board.
- fab.py: ORDER-NOTES rewritten as a friendly request for quotation (LCSC = reference only,
  equivalents welcome, preferences not conditions, terminal direction named); BOM.csv/CPL.csv;
  supplier ACCESSORIES.csv without internal notes or RS-485 items.
- Gates: ERC 0/0; DRC 0 violations / 0 unconnected; pincaps 0 over; analog nets identical to
  the pre-0036 board.

Co-Authored-By: Claude Opus 5.5 <noreply@anthropic.com>
Connections:
- net +24V_RAW: now also J601.3 (Pin_3); no longer J601.1 (Pin_1)
- net CHASSIS: now also J601.1 (Pin_1); no longer J601.3 (Pin_3)
Changed lines of the file:
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@@
 		)
 	)
-	(label "+24V_RAW"
+	(global_label "CHASSIS"
+		(shape bidirectional)
 		(at 25.4 27.94 180)
+		(fields_autoplaced yes)
 		(effects
 			(font
 				(size 1.27 1.27)
 			)
-			(justify right bottom)
+			(justify right)
+		)
+		(property "Intersheetrefs" "${INTERSHEET_REFS}"
+			(at 25.4 27.94 0)
+			(effects
+				(font
+					(size 1.27 1.27)
+				)
+				(hide yes)
+			)
 		)
 	)
@@
 		)
 	)
-	(global_label "CHASSIS"
-		(shape bidirectional)
+	(label "+24V_RAW"
 		(at 25.4 33.02 180)
-		(fields_autoplaced yes)
 		(effects
 			(font
 				(size 1.27 1.27)
 			)
-			(justify right)
-		)
-		(property "Intersheetrefs" "${INTERSHEET_REFS}"
-			(at 25.4 33.02 0)
-			(effects
-				(font
-					(size 1.27 1.27)
-				)
-				(hide yes)
-			)
+			(justify right bottom)
 		)
 	)
