File: hardware/24ch/thermo24.kicad_pcb (KiCad board)
At the start: 4 copper layers, 170 x 145 mm, 466 parts, among them J101 TC CH1-4, J102 TC CH5-8, J201 TC CH9-12, J202 TC CH13-16, J301 TC CH17-20, J302 TC CH21-24, J401 ENGINE REF FEED/SENSE, J501 AVR ISP, J502 LCD 20x4 HEADER, J503 PANEL BUTTONS, J601 24V IN, J701 TRIP C-NO-NC, J702 ALM C-NO-NC, J703 RS485 A B GND, K701 G6K-2F-Y DC5, K702 G6K-2F-Y DC5, Q401 2N7002, Q402 MMBT3906, Q701 2N7002, Q702 2N7002, SW501 UP, SW502 DOWN, SW503 SET, SW504 ESC, SW505 ACK, U101 AD7124-8BCPZ, U102 TMP126DCKR, U103 TMP126DCKR, U201 AD7124-8BCPZ, U202 TMP126DCKR, U203 TMP126DCKR, U301 AD7124-8BCPZ, U302 TMP126DCKR, U303 TMP126DCKR, U401 B0505S-1WR2, U402 LP2985IM5X-3.3, U403 CA-IS3761HW, U404 CA-IS3761HW, U405 CA-IS3761HW, U406 REF3030AIDBZR, U407 MCP6001T-I/OT, U408 TLV7031DBVR, U409 TL431, U501 ATmega1284P-AU, U601 LM5164DDAR, U703 ADM2587EBRWZ, Y501 8MHz

Commit message: 24ch REV A4 (WIP): gated TMP126 SIO driver, PD5 = SIO_WR_N, ESC via diodes
- PD5 (was BTN_ESC) drives SIO_WR_N through spare U405 channel C to U411
  74LVC1G125 (OE); DIN -> U411 -> R446 220R -> DOUT_ISO; R445 10k, R447 100k,
  C421 100n, R439 10k pull-up. R443 22k removed (R446 reuses its footprint).
  Same circuit as hardware/family (fixes the TMP126 SIO edge, 1.2-1.6 us vs 100 ns).
- ESC button kept: D501/D502 1N4148W pull BTN_UP and BTN_DOWN together;
  firmware reads UP+DOWN as ESC.
- Board edited incrementally (delta.py, capnear.py, maze.py with In2 for
  SIO_DRV / SIO_WR_N_ISO); dead DIN branch to the old R443 pad removed.
- Gates: build.py ERC 0 errors 0 warnings, netlist 0 mismatches;
  finish.py DRC (errors, refilled) 0 violations, 0 unconnected; pincaps 0 over
  (U411 added). Silk, full DRC, fab release still to do.
- Title/release names REV A4.

Co-Authored-By: Claude Opus 5.5 <noreply@anthropic.com>
Parts:
- added C421: 100n, Capacitor_SMD:C_0805_2012Metric, F.Cu at (80.3, 117.5)
- added D501: 1N4148W, Diode_SMD:D_SOD-123, F.Cu at (136.9, 54.3)
- added D502: 1N4148W, Diode_SMD:D_SOD-123, F.Cu at (133.3, 53.1)
- added R439: 10k, Resistor_SMD:R_0805_2012Metric, F.Cu at (95.5, 94.1)
- added R445: 10k, Resistor_SMD:R_0805_2012Metric, F.Cu at (82.6, 117.5)
- added R447: 100k, Resistor_SMD:R_0805_2012Metric, F.Cu at (85.4, 111.2)
- added U411: 74LVC1G125, Package_TO_SOT_SMD:SOT-23-5, F.Cu at (81.5, 113.8)
- R446: renamed from R443; value 22k -> 220R
Connections:
- R446 pad 1: DIN_ISO -> /ISOLATION_2/SIO_DRV
- U405 pad 13: unconnected-(U405-OUTC-Pad13) -> SIO_WR_N_ISO
- U405 pad 4: GND -> SIO_WR_N
- U501 pad 14: /MCU/BTN_ESC -> SIO_WR_N
Routing:
- net /MCU/BTN_ESC: track 141.5 -> 52.9 mm, vias 4 -> 2
- net SIO_WR_N: track 0.00 -> 48.3 mm, vias 0 -> 2
- net SIO_WR_N_ISO: track 0.00 -> 26.3 mm, vias 0 -> 5
- net /MCU/BTN_DOWN: track 130.6 -> 141.3 mm, vias 5 -> 6
- net DIN_ISO: track 286.7 -> 277.8 mm, vias 18 -> 16
- net /MCU/BTN_UP: track 114.8 -> 122.5 mm
- net /ISOLATION_2/SIO_DRV: track 0.00 -> 5.26 mm, vias 0 -> 2
- net +3V3_ISO: track 136.9 -> 139.5 mm, vias 98 -> 104
- net GND_ISO: track 172.8 -> 175.0 mm, vias 127 -> 129
- net GND: track 73.6 -> 72.0 mm
- net CS_ADC3_ISO: track 123.1 -> 121.9 mm
- net +5V: track 73.8 -> 74.8 mm, vias 36 -> 39
