File: hardware/24ch/thermo24.kicad_pcb (KiCad board)
At the start: 4 copper layers, 170 x 145 mm, 473 parts, among them J101 TC CH1-4, J102 TC CH5-8, J201 TC CH9-12, J202 TC CH13-16, J301 TC CH17-20, J302 TC CH21-24, J401 ENGINE REF FEED/SENSE, J501 AVR ISP, J502 LCD 20x4 HEADER, J503 PANEL BUTTONS, J601 24V IN, J701 TRIP C-NO-NC, J702 ALM C-NO-NC, J703 RS485 A B GND, K701 G6K-2F-Y DC5, K702 G6K-2F-Y DC5, Q401 2N7002, Q402 MMBT3906, Q701 2N7002, Q702 2N7002, SW501 UP, SW502 DOWN, SW503 SET, SW504 ESC, SW505 ACK, U101 AD7124-8BCPZ, U102 TMP126DCKR, U103 TMP126DCKR, U201 AD7124-8BCPZ, U202 TMP126DCKR, U203 TMP126DCKR, U301 AD7124-8BCPZ, U302 TMP126DCKR, U303 TMP126DCKR, U401 B0505S-1WR2, U402 LP2985IM5X-3.3, U403 CA-IS3761HW, U404 CA-IS3761HW, U405 CA-IS3761HW, U406 REF3030AIDBZR, U407 MCP6001T-I/OT, U408 TLV7031DBVR, U409 TL431, U411 74LVC1G125, U501 ATmega1284P-AU, U601 LM5164DDAR, U703 ADM2587EBRWZ, Y501 8MHz

Commit message: 24ch: clean DRC-dangling tracks (7 overshoots trimmed 0.3-4.7 mm, 3 leftover bits + overlapping DIN_ISO stub removed; 6 junction vias kept), new gen/dangling.py; fab.py adds a warnings DRC pass and blocks on dangling tracks (found by an external kicad-review report; release DRC was --severity-error only)
Co-Authored-By: Claude Opus 5.5 <noreply@anthropic.com>
Routing:
- net CS_ADC3_ISO: track 121.9 -> 113.2 mm
- net SCK: track 91.4 -> 86.8 mm
- net CS_ADC1_ISO: track 195.1 -> 192.1 mm
- net SCLK_ISO: track 336.8 -> 334.2 mm
- net DIN_ISO: track 277.8 -> 276.5 mm
- net /MCU/LCD_D6: track 25.0 -> 24.4 mm
Changed lines of the file:
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@@
 	(segment
 		(start 158.8083 47)
-		(end 158.8083 46.055)
+		(end 158.8083 46.45)
 		(width 0.2)
 		(locked yes)
@@
 	)
 	(segment
-		(start 25.1983 109.663)
+		(start 25.1983 109.35)
 		(end 25.1983 106.655)
 		(width 0.2)
@@
 	)
 	(segment
-		(start 110.15 108.4)
-		(end 110.35 108.6)
-		(width 0.2)
-		(layer "F.Cu")
-		(net "DIN_ISO")
-	)
-	(segment
 		(start 89.45 112.05)
 		(end 89.4 112.1)
@@
 	)
 	(segment
-		(start 110.35 108.6)
-		(end 110.35 108.65)
-		(width 0.2)
-		(layer "F.Cu")
-		(net "DIN_ISO")
-	)
-	(segment
 		(start 86.85 113.25)
 		(end 86.8 113.25)
@@
 	)
 	(segment
-		(start 109.55 107.75)
-		(end 110.15 108.35)
-		(width 0.2)
-		(layer "F.Cu")
-		(net "DIN_ISO")
-	)
-	(segment
 		(start 89.5 112.05)
 		(end 89.45 112.05)
@@
 	)
 	(segment
-		(start 110.35 108.65)
-		(end 110.4 108.7)
-		(width 0.2)
-		(layer "F.Cu")
-		(net "DIN_ISO")
-	)
-	(segment
 		(start 90.2 111.7)
 		(end 90.15 111.75)
@@
 	)
 	(segment
-		(start 110.15 108.35)
-		(end 110.15 108.4)
-		(width 0.2)
-		(layer "F.Cu")
-		(net "DIN_ISO")
-	)
-	(segment
 		(start 86.7 113.3)
 		(end 86.65 113.35)
@@
 	)
 	(segment
-		(start 35.9455 38.2159)
+		(start 36.2148 38.4852)
 		(end 36.5067 38.7771)
 		(width 0.2)
@@
 	(segment
 		(start 64.7668 105.962)
-		(end 61.434 109.295)
+		(end 62.989451 107.739455)
 		(width 0.2)
 		(layer "F.Cu")
@@
 	)
 	(segment
-		(start 22.5 111.2)
+		(start 19.5 111.2)
 		(end 16.95 111.2)
 		(width 0.2)
@@
 	)
 	(segment
-		(start 38.65 81)
-		(end 38.65 80.95)
-		(width 0.2)
-		(layer "F.Cu")
-		(net "CS_CJ6_ISO")
-	)
-	(segment
 		(start 16.2 116.35)
 		(end 16.2 116.3)
@@
 	(segment
 		(start 88.75 38.29)
-		(end 88.75 63.5234)
+		(end 88.75 58.85)
 		(width 0.2)
 		(locked yes)
@@
 	(segment
 		(start 87.48 43)
-		(end 87.48 63.9122)
+		(end 87.48 63.35)
 		(width 0.2)
 		(locked yes)
@@
 		(width 0.2)
 		(layer "B.Cu")
-		(net "CS_ADC3_ISO")
-	)
-	(segment
-		(start 37.25 43.8)
-		(end 37.25 35.15)
-		(width 0.2)
-		(layer "B.Cu")
