File: hardware/24ch/thermo24.kicad_sch (KiCad schematic)
At the start: 10 parts

Commit message: 24ch REV A4: Astra review fixes, release 195548-b4c4e2
Astra (gpt-6-astra, high): no redesign blocker. Fixed its documentation
findings: schematic title REV A4 and RS-485 block no longer called DNP;
ASSEMBLY-SPEC.pdf generated into the release; I-085 now says J601 pin 1 =
CHASSIS, pin 3 = +24V (0036 D7 turn); TMP126 write transactions keep
SIO_WR_N low through data and CRC (0041, c_iso.py note).
ERC 0/0, netlist 0 mismatches, board unchanged (delta dry: 0), release DRC
0/0/0, BOM 96 lines. Previous releases archived in _OLD_DO_NOT_ORDER.

Co-Authored-By: Claude Opus 5.5 <noreply@anthropic.com>
Other:
- title: Thermo 24-channel protection unit - REV A3 -> Thermo 24-channel protection unit - REV A4
Changed lines of the file:
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@@
 	(paper "A3")
 	(title_block
-		(title "Thermo 24-channel protection unit - REV A3")
+		(title "Thermo 24-channel protection unit - REV A4")
 		(company "Thermo 24-ch protection unit")
 		(rev "A3")
