File: hardware/40ch/thermo40.kicad_pcb (KiCad board)
At the start: 4 copper layers, 250 x 145 mm, 731 parts, among them J1001 PT100 1-2 (A B C), J1002 PT100 3 (A B C), J101 TC CH1-4, J102 TC CH5-8, J201 TC CH9-12, J202 TC CH13-16, J301 TC CH17-20, J302 TC CH21-24, J401 ENGINE REF FEED/SENSE, J501 AVR ISP, J502 LCD 20x4 HEADER, J503 PANEL BUTTONS, J601 24V IN, J701 TRIP C-NO-NC, J702 ALM C-NO-NC, J703 RS485 A B GND, J801 TC CH25-28, J802 TC CH29-32, J901 TC CH33-36, J902 TC CH37-40, K701 G6K-2F-Y DC5, K702 G6K-2F-Y DC5, Q401 2N7002, Q402 MMBT3906, Q701 2N7002, Q702 2N7002, SW501 UP, SW502 DOWN, SW503 SET, SW504 ESC, SW505 ACK, U1001 AD7124-8BCPZ, U101 AD7124-8BCPZ, U102 TMP126DCKR, U103 TMP126DCKR, U201 AD7124-8BCPZ, U202 TMP126DCKR, U203 TMP126DCKR, U301 AD7124-8BCPZ, U302 TMP126DCKR, U303 TMP126DCKR, U401 B0505S-1WR2, U402 LP2985IM5X-3.3, U403 CA-IS3761HW, U404 CA-IS3761HW, U406 REF3030AIDBZR, U407 MCP6001T-I/OT, U408 TLV7031DBVR, U409 TL431, U410 74HC154, U411 74LVC1G125, U501 ATmega1284P-AU, U601 LM5164DDAR, U703 ADM2587EBRWZ, U801 AD7124-8BCPZ, U802 TMP126DCKR, U803 TMP126DCKR, U901 AD7124-8BCPZ, U902 TMP126DCKR, U903 TMP126DCKR, Y501 8MHz

Commit message: 40ch, 8ch-new: dangling trims, 8ch-new I-129 relay rule; re-released 141240 / 141437 under the new warning gate; I-129, I-131 closed
40ch: DRC 0/0/0, warnings 3 silk, pincaps 0, holes 0, fill 1212/1212, MANIFEST 76/76.
8ch-new: DRC 0/0/0, warnings silk only, pincaps 0, holes 0, fill 496/496, MANIFEST 56/56.

Co-Authored-By: Claude Opus 5.5 <noreply@anthropic.com>
Routing:
- net SCK: track 91.4 -> 86.8 mm
- net /MCU/LCD_D6: track 25.0 -> 24.4 mm
- net DOUT_ISO: track 515.6 -> 515.1 mm
- net /BANK_D_2/REGCAPD_D: track 4.70 -> 4.99 mm, vias 1 -> 0
- net /BANK_E_2/REGCAPD_E: track 4.70 -> 4.99 mm, vias 1 -> 0
Changed lines of the file:
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@@
 	)
 	(segment
-		(start 33.25 50.65)
-		(end 33.25 50.3)
+		(start 32.6094 53.5726)
+		(end 32.7 53.3)
 		(width 0.2)
-		(locked yes)
 		(layer "F.Cu")
 		(net "/BANK_D_2/REGCAPD_D")
 	)
-	(via
-		(at 32.6094 53.5726)
-		(size 0.6)
-		(drill 0.3)
-		(layers "F.Cu" "B.Cu")
+	(segment
+		(start 33.25 50.65)
+		(end 33.25 50.3)
+		(width 0.2)
 		(locked yes)
+		(layer "F.Cu")
 		(net "/BANK_D_2/REGCAPD_D")
 	)
@@
 	)
 	(segment
+		(start 158.8083 47)
+		(end 158.8083 46.4)
+		(width 0.2)
+		(layer "B.Cu")
+		(net "/OUTPUTS/TRIP_LOW")
+	)
+	(segment
 		(start 145.65 44.35)
 		(end 145.7 44.4)
@@
 	)
 	(segment
-		(start 158.8083 47)
-		(end 158.8083 46.055)
-		(width 0.2)
-		(locked yes)
-		(layer "B.Cu")
-		(net "/OUTPUTS/TRIP_LOW")
-	)
-	(segment
 		(start 156.45 45.45)
 		(end 156.9 45.45)
@@
 	)
 	(segment
-		(start 214 72.65)
-		(end 214 73.5)
-		(width 0.2)
-		(layer "B.Cu")
-		(net "DOUT_ISO")
-	)
-	(segment
 		(start 214.15 82.85)
 		(end 214.15 82.9)
@@
 	)
 	(segment
+		(start 214 72.65)
+		(end 214 73)
+		(width 0.2)
+		(layer "B.Cu")
+		(net "DOUT_ISO")
+	)
+	(segment
 		(start 36.75 81.15)
 		(end 36.65 81.25)
@@
 	)
 	(segment
-		(start 35.9455 38.2159)
-		(end 36.5067 38.7771)
-		(width 0.2)
-		(locked yes)
-		(layer "F.Cu")
-		(net "SCLK_ISO")
-	)
-	(segment
 		(start 33.549999 78.55)
 		(end 33.6 78.55)
@@
 	)
 	(segment
+		(start 36.2148 38.4852)
+		(end 36.5067 38.7771)
+		(width 0.2)
+		(layer "F.Cu")
+		(net "SCLK_ISO")
+	)
+	(segment
 		(start 214.15 89.5)
 		(end 214.15 89.45)
@@
 	)
 	(segment
-		(start 88.75 38.29)
-		(end 88.75 63.5234)
-		(width 0.2)
-		(locked yes)
-		(layer "B.Cu")
-		(net "SCK")
-	)
-	(segment
 		(start 75.3072 74)
 		(end 74.35 73.0428)
@@
 	)
 	(segment
+		(start 88.75 38.29)
+		(end 88.75 58.85)
+		(width 0.2)
+		(layer "B.Cu")
+		(net "SCK")
+	)
+	(segment
 		(start 74.575 95.3097)
 		(end 74.575 89.3099)
@@
 	(segment
 		(start 87.48 43)
-		(end 87.48 63.9122)
+		(end 87.48 63.35)
 		(width 0.2)
-		(locked yes)
 		(layer "B.Cu")
 		(net "/MCU/LCD_D6")
@@
 	)
 	(segment
+		(start 217.3906 72.4274)
+		(end 217.3 72.7)
+		(width 0.2)
+		(layer "F.Cu")
+		(net "/BANK_E_2/REGCAPD_E")
+	)
+	(segment
 		(start 217 74.85)
 		(end 216.95 74.9)
@@
 		(net "/BANK_E_2/REGCAPD_E")
 	)
-	(via
-		(at 217.3906 72.4274)
-		(size 0.6)
-		(drill 0.3)
-		(layers "F.Cu" "B.Cu")
-		(locked yes)
-		(net "/BANK_E_2/REGCAPD_E")
-	)
